Commit message: updated some moveit,but controller failed

File: src/car_witharm/config/gazebo_car2_sld.urdf (robot description, URDF)
Before this commit: robot car2_sld, 13 links, 12 joints
Links:
- added link camera_link; visual box size=0.01 0.1 0.01
- added link laser_link; visual box size=0.01 0.1 0.01
- added link laserholder_link; visual cylinder length=0.8 radius=0.01
- link arm1_link: mass 1.27500464040644 -> 0.1
- link arm2_link: mass 0.930153151725561 -> 0.1
- link arm3_link: mass 1.22106539786534 -> 0.1
- link base_link: mass 164.353963589239 -> 1
- link finger1_link: mass 0.00805 -> 0.01
- link finger2_link: mass 0.00805 -> 0.01
- link hand_link: mass 0.0516505006136003 -> 0.05
- link wlb_link: mass 0.409695097954645 -> 0.4
- link wlf_link: mass 0.409695097954645 -> 0.4
- link wrb_link: mass 0.409695097954645 -> 0.4
- link wrf_link: mass 0.409695097954645 -> 0.4
Joints:
- added joint camera_joint: type fixed, parent base_link, child camera_link, origin xyz=0.3 0 0.01 rpy=0 0 0
- added joint laser_joint: type fixed, parent base_link, child laser_link, origin xyz=-0.35 0 0.805 rpy=0 0 0
- added joint laserholder_joint: type fixed, parent base_link, child laserholder_link, origin xyz=-0.35 0 0.4 rpy=0 0 0
- joint hand_joint: type continuous -> fixed
- joint wlb_joint: axis 0 0 1 -> 0 1 0; origin xyz=-0.325 0.29 -0.02 rpy=1.5707963267949 0 0 -> xyz=-0.325 0.29 -0.02 rpy=0 0 0
- joint wlf_joint: axis 0 0 1 -> 0 1 0; origin xyz=0.325 0.29 -0.02 rpy=1.5708 0 0 -> xyz=0.325 0.29 -0.02 rpy=0 0 0
- joint wrb_joint: axis 0 0 1 -> 0 1 0; origin xyz=-0.325 -0.29 -0.02 rpy=1.5707963267949 0 0 -> xyz=-0.325 -0.29 -0.02 rpy=0 0 0
- joint wrf_joint: axis 0 0 1 -> 0 1 0; origin xyz=0.325 -0.29 -0.02 rpy=1.5708 0 0 -> xyz=0.325 -0.29 -0.02 rpy=0 0 0
