Commit message: 12.17 complete submission

File: src/car2_sld/urdf/car2_sld.urdf (robot description, URDF)
Before this commit: robot car2_sld, 15 links, 14 joints
Joints:
- joint camera_joint: origin xyz=0 0 0.015 rpy=0 0 0 -> xyz=0 0 0.115 rpy=0 0 0; parent laser_link -> base_link

Commit message: navigation a bit

File: src/car2_sld/urdf/car2_sld.urdf (robot description, URDF)
Before this commit: robot car2_sld, 15 links, 14 joints
Joints:
- joint hand_joint: type continuous -> fixed

Commit message: test

File: src/car2_sld/urdf/car2_sld.urdf (robot description, URDF)
Before this commit: robot car2_sld, 15 links, 14 joints
Links:
- added link laserholder_link; visual cylinder length=0.8 radius=0.01
- link arm1_link: mass 1.27500464040644 -> 0.1
- link arm2_link: mass 0.930153151725561 -> 0.1
- link arm3_link: mass 1.22106539786534 -> 0.1
- link base_link: mass 164.353963589239 -> 1
- link finger1_link: mass 0.00805 -> 0.01
- link finger2_link: mass 0.00805 -> 0.01
- link hand_link: mass 0.0516505006136003 -> 0.05
- link wlb_link: mass 0.409695097954645 -> 0.4
- link wlf_link: mass 0.409695097954645 -> 0.4
- link wrb_link: mass 0.409695097954645 -> 0.4
- link wrf_link: mass 0.409695097954645 -> 0.4
Joints:
- added joint laserholder_joint: type fixed, parent base_link, child laserholder_link, origin xyz=-0.35 0 0.4 rpy=0 0 0
- joint camera_joint: origin xyz=0 0 0.115 rpy=0 0 0 -> xyz=0.3 0 0.01 rpy=0 0 0
- joint laser_joint: origin xyz=0.3 0 0.03 rpy=0 0 0 -> xyz=-0.35 0 0.805 rpy=0 0 0

Commit message: updated navigator

File: src/car2_sld/urdf/car2_sld.urdf (robot description, URDF)
Before this commit: robot car2_sld, 16 links, 15 joints
Joints:
- joint wlb_joint: axis 0 0 1 -> 0 1 0; origin xyz=-0.325 0.29 -0.02 rpy=1.5707963267949 0 0 -> xyz=-0.325 0.29 -0.02 rpy=0 0 0
- joint wlf_joint: axis 0 0 1 -> 0 1 0; origin xyz=0.325 0.29 -0.02 rpy=1.5708 0 0 -> xyz=0.325 0.29 -0.02 rpy=0 0 0
- joint wrb_joint: axis 0 0 1 -> 0 1 0; origin xyz=-0.325 -0.29 -0.02 rpy=1.5707963267949 0 0 -> xyz=-0.325 -0.29 -0.02 rpy=0 0 0
- joint wrf_joint: axis 0 0 1 -> 0 1 0; origin xyz=0.325 -0.29 -0.02 rpy=1.5708 0 0 -> xyz=0.325 -0.29 -0.02 rpy=0 0 0

Commit message: updated voice and mediapipe

File: src/car2_sld/urdf/car2_sld.urdf (robot description, URDF)
Before this commit: robot car2_sld, 16 links, 15 joints
Joints:
- joint camera_joint: origin xyz=0.3 0 0.01 rpy=0 0 0 -> xyz=0.4 0 0.01 rpy=0 0 0
